File: LED_Panel/LED_Panel.kicad_pcb (KiCad board)
At the start: 2 copper layers, 65 x 102 mm, 35 parts, among them J1 Conn_01x20_Male

Commit message: changed 1x20 header digikey PN
Changed lines of the file:
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@@
     (fp_line (start -3.15 1.6) (end -3.15 -1.6) (layer "F.Fab") (width 0.1))
     (fp_line (start 3.15 -1.6) (end 3.15 1.6) (layer "F.Fab") (width 0.1))
-    (pad "1" smd roundrect (at -2.9625 0 270) (size 1.225 3.35) (layers "F.Cu" "F.Paste" "F.Mask") (roundrect_rratio 0.204082)
+    (pad "1" smd roundrect (at -2.9625 0 270) (size 1.225 3.35) (layers "F.Cu" "F.Paste" "F.Mask") (roundrect_rratio 0.2040816327)
       (net 24 "Net-(J1-Pad15)") (pintype "passive"))
-    (pad "2" smd roundrect (at 2.9625 0 270) (size 1.225 3.35) (layers "F.Cu" "F.Paste" "F.Mask") (roundrect_rratio 0.204082)
+    (pad "2" smd roundrect (at 2.9625 0 270) (size 1.225 3.35) (layers "F.Cu" "F.Paste" "F.Mask") (roundrect_rratio 0.2040816327)
       (net 7 "/SEGMENT_3") (pintype "passive"))
     (model "${KICAD6_3DMODEL_DIR}/Resistor_SMD.3dshapes/R_2512_6332Metric.wrl"
@@
     (fp_line (start -3.15 -1.6) (end 3.15 -1.6) (layer "F.Fab") (width 0.1))
     (fp_line (start 3.15 1.6) (end -3.15 1.6) (layer "F.Fab") (width 0.1))
-    (pad "1" smd roundrect (at -2.9625 0 270) (size 1.225 3.35) (layers "F.Cu" "F.Paste" "F.Mask") (roundrect_rratio 0.204082)
+    (pad "1" smd roundrect (at -2.9625 0 270) (size 1.225 3.35) (layers "F.Cu" "F.Paste" "F.Mask") (roundrect_rratio 0.2040816327)
       (net 25 "Net-(J1-Pad11)") (pintype "passive"))
-    (pad "2" smd roundrect (at 2.9625 0 270) (size 1.225 3.35) (layers "F.Cu" "F.Paste" "F.Mask") (roundrect_rratio 0.204082)
+    (pad "2" smd roundrect (at 2.9625 0 270) (size 1.225 3.35) (layers "F.Cu" "F.Paste" "F.Mask") (roundrect_rratio 0.2040816327)
       (net 4 "/SEGMENT_5") (pintype "passive"))
     (model "${KICAD6_3DMODEL_DIR}/Resistor_SMD.3dshapes/R_2512_6332Metric.wrl"
@@
     (fp_line (start 3.15 -1.6) (end 3.15 1.6) (layer "F.Fab") (width 0.1))
     (fp_line (start -3.15 -1.6) (end 3.15 -1.6) (layer "F.Fab") (width 0.1))
-    (pad "1" smd roundrect (at -2.9625 0 90) (size 1.225 3.35) (layers "F.Cu" "F.Paste" "F.Mask") (roundrect_rratio 0.204082)
+    (pad "1" smd roundrect (at -2.9625 0 90) (size 1.225 3.35) (layers "F.Cu" "F.Paste" "F.Mask") (roundrect_rratio 0.2040816327)
       (net 21 "Net-(J1-Pad1)") (pintype "passive"))
-    (pad "2" smd roundrect (at 2.9625 0 90) (size 1.225 3.35) (layers "F.Cu" "F.Paste" "F.Mask") (roundrect_rratio 0.204082)
+    (pad "2" smd roundrect (at 2.9625 0 90) (size 1.225 3.35) (layers "F.Cu" "F.Paste" "F.Mask") (roundrect_rratio 0.2040816327)
       (net 10 "/SEGMENT_8A") (pintype "passive"))
     (model "${KICAD6_3DMODEL_DIR}/Resistor_SMD.3dshapes/R_2512_6332Metric.wrl"
@@
     (fp_line (start 3.15 1.6) (end -3.15 1.6) (layer "F.Fab") (width 0.1))
     (fp_line (start -3.15 -1.6) (end 3.15 -1.6) (layer "F.Fab") (width 0.1))
-    (pad "1" smd roundrect (at -2.9625 0 90) (size 1.225 3.35) (layers "F.Cu" "F.Paste" "F.Mask") (roundrect_rratio 0.204082)
+    (pad "1" smd roundrect (at -2.9625 0 90) (size 1.225 3.35) (layers "F.Cu" "F.Paste" "F.Mask") (roundrect_rratio 0.2040816327)
       (net 22 "Net-(J1-Pad16)") (pintype "passive"))
-    (pad "2" smd roundrect (at 2.9625 0 90) (size 1.225 3.35) (layers "F.Cu" "F.Paste" "F.Mask") (roundrect_rratio 0.204082)
+    (pad "2" smd roundrect (at 2.9625 0 90) (size 1.225 3.35) (layers "F.Cu" "F.Paste" "F.Mask") (roundrect_rratio 0.2040816327)
       (net 5 "/SEGMENT_2") (pintype "passive"))
     (model "${KICAD6_3DMODEL_DIR}/Resistor_SMD.3dshapes/R_2512_6332Metric.wrl"
@@
     (fp_line (start -3.15 1.6) (end -3.15 -1.6) (layer "F.Fab") (width 0.1))
     (fp_line (start 3.15 1.6) (end -3.15 1.6) (layer "F.Fab") (width 0.1))
-    (pad "1" smd roundrect (at -2.9625 0 270) (size 1.225 3.35) (layers "F.Cu" "F.Paste" "F.Mask") (roundrect_rratio 0.204082)
+    (pad "1" smd roundrect (at -2.9625 0 270) (size 1.225 3.35) (layers "F.Cu" "F.Paste" "F.Mask") (roundrect_rratio 0.2040816327)
       (net 26 "Net-(J1-Pad2)") (pintype "passive"))
-    (pad "2" smd roundrect (at 2.9625 0 270) (size 1.225 3.35) (layers "F.Cu" "F.Paste" "F.Mask") (roundrect_rratio 0.204082)
+    (pad "2" smd roundrect (at 2.9625 0 270) (size 1.225 3.35) (layers "F.Cu" "F.Paste" "F.Mask") (roundrect_rratio 0.2040816327)
       (net 12 "/SEGMENT_8B") (pintype "passive"))
     (model "${KICAD6_3DMODEL_DIR}/Resistor_SMD.3dshapes/R_2512_6332Metric.wrl"
@@
     (fp_line (start -3.15 -1.6) (end 3.15 -1.6) (layer "F.Fab") (width 0.1))
     (fp_line (start 3.15 -1.6) (end 3.15 1.6) (layer "F.Fab") (width 0.1))
-    (pad "1" smd roundrect (at -2.9625 0 270) (size 1.225 3.35) (layers "F.Cu" "F.Paste" "F.Mask") (roundrect_rratio 0.204082)
+    (pad "1" smd roundrect (at -2.9625 0 270) (size 1.225 3.35) (layers "F.Cu" "F.Paste" "F.Mask") (roundrect_rratio 0.2040816327)
       (net 27 "Net-(J1-Pad19)") (pintype "passive"))
-    (pad "2" smd roundrect (at 2.9625 0 270) (size 1.225 3.35) (layers "F.Cu" "F.Paste" "F.Mask") (roundrect_rratio 0.204082)
+    (pad "2" smd roundrect (at 2.9625 0 270) (size 1.225 3.35) (layers "F.Cu" "F.Paste" "F.Mask") (roundrect_rratio 0.2040816327)
       (net 14 "/SEGMENT_1B") (pintype "passive"))
     (model "${KICAD6_3DMODEL_DIR}/Resistor_SMD.3dshapes/R_2512_6332Metric.wrl"
@@
     (fp_line (start -3.15 1.6) (end -3.15 -1.6) (layer "F.Fab") (width 0.1))
     (fp_line (start 3.15 1.6) (end -3.15 1.6) (layer "F.Fab") (width 0.1))
-    (pad "1" smd roundrect (at -2.9625 0 270) (size 1.225 3.35) (layers "F.Cu" "F.Paste" "F.Mask") (roundrect_rratio 0.204082)
+    (pad "1" smd roundrect (at -2.9625 0 270) (size 1.225 3.35) (layers "F.Cu" "F.Paste" "F.Mask") (roundrect_rratio 0.2040816327)
       (net 29 "Net-(J1-Pad7)") (pintype "passive"))
-    (pad "2" smd roundrect (at 2.9625 0 270) (size 1.225 3.35) (layers "F.Cu" "F.Paste" "F.Mask") (roundrect_rratio 0.204082)
+    (pad "2" smd roundrect (at 2.9625 0 270) (size 1.225 3.35) (layers "F.Cu" "F.Paste" "F.Mask") (roundrect_rratio 0.2040816327)
       (net 6 "/SEGMENT_6") (pintype "passive"))
     (model "${KICAD6_3DMODEL_DIR}/Resistor_SMD.3dshapes/R_2512_6332Metric.wrl"
@@
     (fp_line (start -3.15 -1.6) (end 3.15 -1.6) (layer "F.Fab") (width 0.1))
     (fp_line (start -3.15 1.6) (end -3.15 -1.6) (layer "F.Fab") (width 0.1))
-    (pad "1" smd roundrect (at -2.9625 0 90) (size 1.225 3.35) (layers "F.Cu" "F.Paste" "F.Mask") (roundrect_rratio 0.204082)
+    (pad "1" smd roundrect (at -2.9625 0 90) (size 1.225 3.35) (layers "F.Cu" "F.Paste" "F.Mask") (roundrect_rratio 0.2040816327)
       (net 28 "Net-(J1-Pad6)") (pintype "passive"))
-    (pad "2" smd roundrect (at 2.9625 0 90) (size 1.225 3.35) (layers "F.Cu" "F.Paste" "F.Mask") (roundrect_rratio 0.204082)
+    (pad "2" smd roundrect (at 2.9625 0 90) (size 1.225 3.35) (layers "F.Cu" "F.Paste" "F.Mask") (roundrect_rratio 0.2040816327)
       (net 9 "/SEGMENT_7") (pintype "passive"))
     (model "${KICAD6_3DMODEL_DIR}/Resistor_SMD.3dshapes/R_2512_6332Metric.wrl"
@@
     (fp_line (start 3.15 1.6) (end -3.15 1.6) (layer "F.Fab") (width 0.1))
     (fp_line (start -3.15 1.6) (end -3.15 -1.6) (layer "F.Fab") (width 0.1))
-    (pad "1" smd roundrect (at -2.9625 0 90) (size 1.225 3.35) (layers "F.Cu" "F.Paste" "F.Mask") (roundrect_rratio 0.204082)
+    (pad "1" smd roundrect (at -2.9625 0 90) (size 1.225 3.35) (layers "F.Cu" "F.Paste" "F.Mask") (roundrect_rratio 0.2040816327)
       (net 23 "Net-(J1-Pad12)") (pintype "passive"))
-    (pad "2" smd roundrect (at 2.9625 0 90) (size 1.225 3.35) (layers "F.Cu" "F.Paste" "F.Mask") (roundrect_rratio 0.204082)
+    (pad "2" smd roundrect (at 2.9625 0 90) (size 1.225 3.35) (layers "F.Cu" "F.Paste" "F.Mask") (roundrect_rratio 0.2040816327)
       (net 31 "/SEGMENT_4") (pintype "passive"))
     (model "${KICAD6_3DMODEL_DIR}/Resistor_SMD.3dshapes/R_2512_6332Metric.wrl"
@@
     (fp_line (start 3.15 1.6) (end -3.15 1.6) (layer "F.Fab") (width 0.1))
     (fp_line (start 3.15 -1.6) (end 3.15 1.6) (layer "F.Fab") (width 0.1))
-    (pad "1" smd roundrect (at -2.9625 0 90) (size 1.225 3.35) (layers "F.Cu" "F.Paste" "F.Mask") (roundrect_rratio 0.204082)
+    (pad "1" smd roundrect (at -2.9625 0 90) (size 1.225 3.35) (layers "F.Cu" "F.Paste" "F.Mask") (roundrect_rratio 0.2040816327)
       (net 30 "Net-(J1-Pad20)") (pintype "passive"))
-    (pad "2" smd roundrect (at 2.9625 0 90) (size 1.225 3.35) (layers "F.Cu" "F.Paste" "F.Mask") (roundrect_rratio 0.204082)
+    (pad "2" smd roundrect (at 2.9625 0 90) (size 1.225 3.35) (layers "F.Cu" "F.Paste" "F.Mask") (roundrect_rratio 0.2040816327)
       (net 13 "/SEGMENT_1A") (pintype "passive"))
     (model "${KICAD6_3DMODEL_DIR}/Resistor_SMD.3dshapes/R_2512_6332Metric.wrl"

Commit message: edited header PN
Other:
- board text added: "https://github.com/wszeto9/ 8-Segment-Numeric-Display"
Changed lines of the file:
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@@
     (thickness 1.6)
   )
-  (paper "A4")
+  (paper "USLetter")
+  (title_block
+    (date "2023-02-08")
+    (rev "A")
+  )
   (layers
     (0 "F.Cu" signal)
@@
     (descr "Harwin Male Horizontal Surface Mount Single Row 2.54mm (0.1 inch) Pitch PCB Connector, M20-89020xx, 20 Pins per row (https://cdn.harwin.com/pdfs/M20-890.pdf), generated with kicad-footprint-generator")
     (tags "connector Harwin M20-890 horizontal")
-    (property "Digikey" "https://www.digikey.com/en/products/detail/sullins-connector-solutions/GEC36SBSN-M89/862247")
+    (property "Digikey" "S1113E-20-ND")
     (property "Sheetfile" "LED_Panel.kicad_sch")
     (property "Sheetname" "")
@@
     (effects (font (size 1 1) (thickness 0.15)))
   )
-  (dimension (type aligned) (layer "F.SilkS")
-    (pts (xy 139 160) (xy 73.999999 160))
-    (height -11.4)
-    (gr_text "65.0000 mm" (at 106.5 170.25) (layer "F.SilkS")
-      (effects (font (size 1 1) (thickness 0.15)))
-    )
-    (format (units 3) (units_format 1) (precision 4))
+  (gr_text "https://github.com/wszeto9/\n8-Segment-Numeric-Display" (at 106.5 149.2) (layer "F.SilkS")
+    (effects (font (size 1 1) (thickness 0.15)))
+  )
+  (dimension (type aligned) (layer "Dwgs.User")
+    (pts (xy 78 157) (xy 78 161))
+    (height 7)
+    (gr_text "2x4.0 mm" (at 66.2 158.9) (layer "Dwgs.User")
+      (effects (font (size 1 1) (thickness 0.15)))
+    )
+    (format (prefix "2x") (units 3) (units_format 1) (precision 1))
+    (style (thickness 0.15) (arrow_length 1.27) (text_position_mode 2) (extension_height 0.58642) (extension_offset 0.5))
+  )
+  (dimension (type aligned) (layer "Dwgs.User")
+    (pts (xy 78 157) (xy 74 157))
+    (height -12)
+    (gr_text "2x4.0 mm" (at 83.1 169) (layer "Dwgs.User")
+      (effects (font (size 1 1) (thickness 0.15)))
+    )
+    (format (prefix "2x") (units 3) (units_format 1) (precision 1))
+    (style (thickness 0.15) (arrow_length 1.27) (text_position_mode 2) (extension_height 0.58642) (extension_offset 0.5) keep_text_aligned)
+  )
+  (dimension (type aligned) (layer "Dwgs.User")
+    (pts (xy 135 157) (xy 78 157))
+    (height -18.1)
+    (gr_text "(57.0 mm)" (at 106.5 173.95) (layer "Dwgs.User")
+      (effects (font (size 1 1) (thickness 0.15)))
+    )
+    (format (prefix "(") (suffix ")") (units 3) (units_format 1) (precision 1))
     (style (thickness 0.15) (arrow_length 1.27) (text_position_mode 0) (extension_height 0.58642) (extension_offset 0.5) keep_text_aligned)
+  )
+  (dimension (type aligned) (layer "Dwgs.User")
+    (pts (xy 73.999999 160) (xy 139 160))
+    (height 20.8)
+    (gr_text "65.0 mm" (at 106.499999 179.65) (layer "Dwgs.User")
+      (effects (font (size 1 1) (thickness 0.15)))
+    )
+    (format (units 3) (units_format 1) (precision 1))
+    (style (thickness 0.15) (arrow_length 1.27) (text_position_mode 0) (extension_height 0.58642) (extension_offset 0.5) keep_text_aligned)
+  )
+  (dimension (type aligned) (layer "Dwgs.User")
+    (pts (xy 81 65) (xy 132 65))
+    (height -10.1)
+    (gr_text "(51.0 mm)" (at 106.5 53.75) (layer "Dwgs.User")
+      (effects (font (size 1 1) (thickness 0.15)))
+    )
+    (format (prefix "(") (suffix ")") (units 3) (units_format 1) (precision 1))
+    (style (thickness 0.15) (arrow_length 1.27) (text_position_mode 0) (extension_height 0.58642) (extension_offset 0.5) keep_text_aligned)
+  )
+  (dimension (type aligned) (layer "Dwgs.User")
+    (pts (xy 81 65) (xy 81 59))
+    (height -10.6)
+    (gr_text "2x6.0 mm" (at 65.5 62) (layer "Dwgs.User")
+      (effects (font (size 1 1) (thickness 0.15)))
+    )
+    (format (prefix "2x") (units 3) (units_format 1) (precision 1))
+    (style (thickness 0.15) (arrow_length 1.27) (text_position_mode 2) (extension_height 0.58642) (extension_offset 0.5))
+  )
+  (dimension (type aligned) (layer "Dwgs.User")
+    (pts (xy 81 65) (xy 74 65))
+    (height 10.276094)
+    (gr_text "2x7.0 mm" (at 77.5 52.7) (layer "Dwgs.User")
+      (effects (font (size 1 1) (thickness 0.15)))
+    )
+    (format (prefix "2x") (units 3) (units_format 1) (precision 1))
+    (style (thickness 0.15) (arrow_length 1.27) (text_position_mode 2) (extension_height 0.58642) (extension_offset 0.5) keep_text_aligned)
+  )
+  (dimension (type aligned) (layer "Dwgs.User")
+    (pts (xy 78 157) (xy 77.95 65))
+    (height -22.051322)
+    (gr_text "(2x92.0 mm)" (at 62 111) (layer "Dwgs.User")
+      (effects (font (size 1 1) (thickness 0.15)))
+    )
+    (format (prefix "(2x") (suffix ")") (units 3) (units_format 1) (precision 1))
+    (style (thickness 0.15) (arrow_length 1.27) (text_position_mode 2) (extension_height 0.58642) (extension_offset 0.5))
+  )
+  (dimension (type aligned) (layer "Dwgs.User")
+    (pts (xy 74.999999 161) (xy 75 59))
+    (height -23.899999)
+    (gr_text "102.0 mm" (at 45.7 110.8) (layer "Dwgs.User")
+      (effects (font (size 1 1) (thickness 0.15)))
+    )
+    (format (units 3) (units_format 1) (precision 1))
+    (style (thickness 0.15) (arrow_length 1.27) (text_position_mode 2) (extension_height 0.58642) (extension_offset 0.5))
   )
   (segment (start 109.875978 66.625) (end 112.150978 68.9) (width 1) (layer "F.Cu") (net 1))
@@
     (polygon
       (pts
-        (xy 168.5 60)
-        (xy 161.5 165.5)
-        (xy 48.5 161)
-        (xy 54 56.5)
+        (xy 138.9 59)
+        (xy 139 160.9)
+        (xy 74 161)
+        (xy 74 59)
       )
     )
