File: LED_Panel/LED_Panel.kicad_sch (KiCad schematic)
At the start: 35 parts, among them J1 Conn_01x20_Male

Commit message: changed 1x20 header digikey PN
Parts:
- J1: Digikey https://www.digikey.com/en/products/detail/sullins-connecto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 -> S1113E-20-ND
Changed lines of the file:
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@@
       (effects (font (size 1.27 1.27)) hide)
     )
-    (property "Digikey" "https://www.digikey.com/en/products/detail/sullins-connector-solutions/GEC36SBSN-M89/862247" (id 4) (at 28.575 160.02 0)
+    (property "Digikey" "S1113E-20-ND" (id 4) (at 28.575 160.02 0)
       (effects (font (size 1.27 1.27)) hide)
     )

Commit message: edited header PN
Other:
- note added: "CHANGELOG/NOTES REV A: Initial Design"
- note added: "Mounting Holes"
- note removed: "CHANGELOG/NOTES REV A:"
- company: (none) -> Winnie Szeto
- moved on the sheet: D1, D10, D11, D12, D13, D14, D15, D16, D17, D18, D19, D2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
