File: LED_Panel_Controller/LED_Panel_Controller.kicad_pcb (KiCad board)
At the start: 2 copper layers, 75 x 32 mm, 37 parts, among them J1 DOUT, J2 DIN, J3 Conn_01x04, J4 Conn_01x20_Female, U1 74HC595, U10 LM2596S-ADJ, U2 AO3400A, U3 AO3400A, U4 AO3400A, U5 AO3400A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

Commit message: updated BOM
Parts:
- J3: value Conn_01x04 -> JST PA
- R2: value 0805,0 -> DNP
Changed lines of the file:
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@@
     (descr "Resistor SMD 0805 (2012 Metric), square (rectangular) end terminal, IPC_7351 nominal, (Body size source: IPC-SM-782 page 72, https://www.pcb-3d.com/wordpress/wp-content/uploads/ipc-sm-782a_amendment_1_and_2.pdf), generated with kicad-footprint-generator")
     (tags "resistor")
-    (property "LCSC" "C17477")
-    (property "MFG" "UNI-ROYAL(Uniroyal Elec)")
-    (property "MFGPN" "0805W8F0000T5E")
+    (property "LCSC" "")
+    (property "MFG" "")
+    (property "MFGPN" "")
     (property "Sheetfile" "LED_Panel_Controller.kicad_sch")
     (property "Sheetname" "")
@@
       (effects (font (size 0.8 0.8) (thickness 0.12)))
     )
-    (fp_text value "0805,0" (at 0 1.65 90) (layer "F.Fab")
+    (fp_text value "DNP" (at 0 1.65 90) (layer "F.Fab")
       (effects (font (size 1 1) (thickness 0.15)))
     )
@@
       (effects (font (size 0.8 0.8) (thickness 0.12)))
     )
-    (fp_text value "Conn_01x04" (at 9.80575 4.51537) (layer "F.Fab")
+    (fp_text value "JST PA " (at 9.80575 4.51537) (layer "F.Fab")
       (effects (font (size 1.000079 1.000079) (thickness 0.15)))
     )

Commit message: changed page size, BOM
Other:
- board text added: "4x M2 Hole"
- board text added: "github.com/wszeto9/8-Segment-Numeric-Display"
Changed lines of the file:
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@@
     (thickness 1.6)
   )
-  (paper "A4")
+  (paper "USLetter")
+  (title_block
+    (date "2023-02-08")
+    (rev "A")
+  )
   (layers
     (0 "F.Cu" signal)
@@
     (descr "Through hole angled socket strip, 1x20, 2.54mm pitch, 8.51mm socket length, single row (from Kicad 4.0.7), script generated")
     (tags "Through hole angled socket strip THT 1x20 2.54mm single row")
-    (property "Digikey" "https://www.amazon.com/Yohii-Female-Header-2-54mm-Connector/dp/B07P1R9CGT/ref=sr_1_2?crid=24L21ACA4OHBU&keywords=female+header+right+angle&qid=1675869501&sprefix=female+header+right+angle%2Caps%2C90&sr=8-2")
+    (property "Digikey" "https://www.amazon.com/Yohii-Female-Header-2-54mm-Connector/dp/B07P1R9CGT/")
     (property "Sheetfile" "LED_Panel_Controller.kicad_sch")
     (property "Sheetname" "")
@@
     (descr "TO-263 / D2PAK / DDPAK SMD package, http://www.infineon.com/cms/en/product/packages/PG-TO263/PG-TO263-5-1/")
     (tags "D2PAK DDPAK TO-263 D2PAK-5 TO-263-5 SOT-426")
-    (property "Digikey" "4518-LM2596S-ADJCT-ND")
+    (property "Digikey" "https://www.amazon.com/gp/product/B0B63GQDJW/")
     (property "MFGPN" "LM2596S-ADJ")
     (property "Sheetfile" "LED_Voltage_buck.kicad_sch")
@@
     (effects (font (size 0.8 0.8) (thickness 0.12)) (justify left mirror))
   )
+  (gr_text "github.com/wszeto9/8-Segment-Numeric-Display" (at 116.7 74.6) (layer "B.SilkS")
+    (effects (font (size 1 1) (thickness 0.15)) (justify mirror))
+  )
   (gr_text "Jump R2 if\nVin=7V/2A" (at 143.9 72.4) (layer "F.SilkS")
     (effects (font (size 0.8 0.8) (thickness 0.12)))
@@
   (gr_text "GND|+VIN" (at 142.9 88.3) (layer "F.SilkS")
     (effects (font (size 1 1) (thickness 0.15)))
+  )
+  (gr_text "4x M2 Hole" (at 73.9 100.45) (layer "Dwgs.User")
+    (effects (font (size 1 1) (thickness 0.15)))
+  )
+  (dimension (type aligned) (layer "Dwgs.User")
+    (pts (xy 79 97.5) (xy 154 97.5))
+    (height 7.599999)
+    (gr_text "75.0000 mm" (at 116.5 103.949999) (layer "Dwgs.User")
+      (effects (font (size 1 1) (thickness 0.15)))
+    )
+    (format (units 3) (units_format 1) (precision 4))
+    (style (thickness 0.15) (arrow_length 1.27) (text_position_mode 0) (extension_height 0.58642) (extension_offset 0.5) keep_text_aligned)
+  )
+  (dimension (type aligned) (layer "Dwgs.User")
+    (pts (xy 80 98.5) (xy 80 66.5))
+    (height -12.95)
+    (gr_text "32.0 mm" (at 62.9 82.35) (layer "Dwgs.User")
+      (effects (font (size 1 1) (thickness 0.15)))
+    )
+    (format (units 3) (units_format 1) (precision 1))
+    (style (thickness 0.15) (arrow_length 1.27) (text_position_mode 2) (extension_height 0.58642) (extension_offset 0.5))
+  )
+  (dimension (type aligned) (layer "Dwgs.User")
+    (pts (xy 81.25 96.25) (xy 79 96.25))
+    (height -4.95)
+    (gr_text "4x2.25 mm" (at 85.9 101.15) (layer "Dwgs.User")
+      (effects (font (size 1 1) (thickness 0.15)))
+    )
+    (format (prefix "4x") (units 3) (units_format 1) (precision 2))
+    (style (thickness 0.15) (arrow_length 1) (text_position_mode 2) (extension_height 0.58642) (extension_offset 0.3) keep_text_aligned)
+  )
+  (dimension (type aligned) (layer "Dwgs.User")
+    (pts (xy 81.25 96.25) (xy 81.25 98.5))
+    (height 3.55)
+    (gr_text "4x2.25 mm" (at 72.5 97.1) (layer "Dwgs.User")
+      (effects (font (size 1 1) (thickness 0.15)))
+    )
+    (format (prefix "4x") (units 3) (units_format 1) (precision 2))
+    (style (thickness 0.15) (arrow_length 1) (text_position_mode 2) (extension_height 0.58642) (extension_offset 0.3))
   )
   (segment (start 90.82 69.5) (end 88.5 69.5) (width 1) (layer "F.Cu") (net 1))
@@
     (polygon
       (pts
-        (xy 164.25 107.75)
-        (xy 69.5 103)
-        (xy 68 55)
-        (xy 166 54.5)
+        (xy 154 98.5)
+        (xy 79 98.5)
+        (xy 79 66.5)
+        (xy 154 66.5)
       )
     )
