File: LED_Panel_Controller/LED_Panel_Controller.kicad_sch (KiCad schematic)
At the start: 26 parts, among them J1 DOUT, J2 DIN, J3 Conn_01x04, J4 Conn_01x20_Female, U1 74HC595, U2 AO3400A, U3 AO3400A, U4 AO3400A, U5 AO3400A, U6 AO3400A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

Commit message: updated BOM
Parts:
- J3: value Conn_01x04 -> JST PA
- R2: value 0805,0 -> DNP; LCSC C17477 -> (none); MFG UNI-ROYAL(Uniroyal Elec) -> (none); MFGPN 0805W8F0000T5E -> (none)
Other:
- note added: "CHANGELOG/NOTES REV A: Initial Commit"
- note added: "Mounting Hole"
- note added: "Output header to LED Panel"
- note added: "Power Input with Polyfuse"
- note added: "Power Rail Indicators"
- note removed: "CHANGELOG/NOTES REV A:"
- moved on the sheet: C6, D2, D3, D4, F1, H1, H2, H3, H4, J1, J2, J3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

Commit message: changed page size, BOM
Parts:
- J4: Digikey https://www.amazon.com/Yohii-Female-Header-2-54mm-Connector/dp/B07P1R9CGT/ref=sr_1_2?crid=24L21ACA4OHBU&keywords=female+header+right+angle&qid=1675869501&sprefix=female+header+right+angle%2Caps%2C90&sr=8-2 -> https://www.amazon.com/Yohii-Female-Header-2-54mm-Connector/dp/B07P1R9CGT/
Changed lines of the file:
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@@
       (effects (font (size 1.27 1.27)) hide)
     )
-    (property "Digikey" "https://www.amazon.com/Yohii-Female-Header-2-54mm-Connector/dp/B07P1R9CGT/ref=sr_1_2?crid=24L21ACA4OHBU&keywords=female+header+right+angle&qid=1675869501&sprefix=female+header+right+angle%2Caps%2C90&sr=8-2" (id 4) (at 135.89 165.735 0)
+    (property "Digikey" "https://www.amazon.com/Yohii-Female-Header-2-54mm-Connector/dp/B07P1R9CGT/" (id 4) (at 135.89 165.735 0)
       (effects (font (size 1.27 1.27)) hide)
     )
